File: discipline-pcb.kicad_pcb (KiCad board)
At the start: 2 copper layers, 304.9 x 122.8 mm, 180 parts, among them J1 AVR-ISP-6, SW1 KEYSW, SW10 KEYSW, SW11 KEYSW, SW12 KEYSW, SW13 KEYSW, SW14 KEYSW, SW15 KEYSW, SW16 KEYSW, SW17 KEYSW, SW18 KEYSW, SW19 KEYSW, SW2 KEYSW, SW20 KEYSW, SW21 KEYSW, SW22 KEYSW, SW23 KEYSW, SW24 KEYSW, SW25 KEYSW, SW26 KEYSW, SW27 KEYSW, SW28 KEYSW, SW29 KEYSW, SW3 KEYSW, SW30 KEYSW, SW31 KEYSW, SW32 KEYSW, SW33 KEYSW, SW34 KEYSW, SW35 KEYSW, SW36 KEYSW, SW37 KEYSW, SW38 KEYSW, SW39 KEYSW, SW4 KEYSW, SW40 KEYSW, SW41 KEYSW, SW42 KEYSW, SW43 KEYSW, SW44 KEYSW, SW45 KEYSW, SW46 KEYSW, SW47 KEYSW, SW48 KEYSW, SW49 KEYSW, SW5 KEYSW, SW50 KEYSW, SW51 KEYSW, SW52 KEYSW, SW53 KEYSW, SW54 KEYSW, SW55 KEYSW, SW56 KEYSW, SW57 KEYSW, SW58 KEYSW, SW59 KEYSW, SW6 KEYSW, SW60 KEYSW, SW61 KEYSW, SW62 KEYSW, SW63 KEYSW, SW64 KEYSW, SW65 KEYSW, SW66 KEYSW, SW67 KEYSW, SW68 KEYSW, SW69 KEYSW, SW7 KEYSW, SW70 KEYSW, SW71 KEYSW, SW72 KEYSW, SW73 KEYSW, SW74 KEYSW, SW8 KEYSW, SW9 KEYSW, U1 ATmega32A-PU, Y1 Crystal

Commit message: hopefully made it ISO compatible
Parts:
- added D75: , cftkb:D_DO-35_SOD27_P5.08mm_Horizontal, F.Cu at (85.8, 125.8)
- added SW75: KEYSW, cftkb:SW_Cherry_MX1A_1.00u_PCB-NOSCREEN, F.Cu at (96.5, 142.1)
- added SWb29: KEYSW, MX_Only:MXOnly-ISO-ROTATED-ReversedStabilizers-NoLED, F.Cu at (334.4, 118.7)
- added SWb43: KEYSW, cftkb:SW_Cherry_MX1A_1.00u_PCB-NOSCREEN, F.Cu at (315.5, 123.0)
- added SWb45: KEYSW, cftkb:SW_Cherry_MX1A_1.25u_PCBNOSCREEN, F.Cu at (75.0, 142.1)
- C1, C2: footprint cftkb:C_Disc_D3.0mm_W1.6mm_P2.50mm -> cftkb:D_DO-35_SOD27_P5.08mm_Horizontal
- C3: footprint cftkb:CP_Radial_D4.0mm_P1.50mm -> cftkb:D_DO-35_SOD27_P5.08mm_Horizontal
- C4, C5: footprint cftkb:C_Disc_D4.3mm_W1.9mm_P5.00mm -> cftkb:D_DO-35_SOD27_P5.08mm_Horizontal
- SW63, SW64: footprint cftkb:SW_Cherry_MX1A_1.00u_PCB-NOSCREEN -> cftkb:SW_Cherry_MX1A_1.25u_PCBNOSCREEN
Routing:
- net row3: track 287.2 -> 361.1 mm, vias 3 -> 5
- net Net-(D29-Pad2): track 117.7 -> 139.3 mm, vias 0 -> 1
- net Net-(D75-Pad2): track 0.00 -> 16.4 mm
- net col13: track 146.9 -> 162.0 mm
- net Net-(D43-Pad2): track 140.6 -> 152.5 mm
- net Net-(D45-Pad2): track 76.5 -> 86.0 mm
- net col0: track 355.0 -> 364.5 mm
- net col12: track 182.7 -> 187.9 mm
- net Net-(D56-Pad2): track 145.3 -> 147.3 mm
Other:
- board text added: "coseyfannitutti 2019 rev1 messed with by bcopping"
- board text removed: "coseyfannitutti 2019 rev1"
