File: discipline-pcb.kicad_pcb (KiCad board)
At the start: 2 copper layers, 304.9 x 122.8 mm, 185 parts, among them J1 AVR-ISP-6, SW1 KEYSW, SW10 KEYSW, SW11 KEYSW, SW12 KEYSW, SW13 KEYSW, SW14 KEYSW, SW15 KEYSW, SW16 KEYSW, SW17 KEYSW, SW18 KEYSW, SW19 KEYSW, SW2 KEYSW, SW20 KEYSW, SW21 KEYSW, SW22 KEYSW, SW23 KEYSW, SW24 KEYSW, SW25 KEYSW, SW26 KEYSW, SW27 KEYSW, SW28 KEYSW, SW29 KEYSW, SW3 KEYSW, SW30 KEYSW, SW31 KEYSW, SW32 KEYSW, SW33 KEYSW, SW34 KEYSW, SW35 KEYSW, SW36 KEYSW, SW37 KEYSW, SW38 KEYSW, SW39 KEYSW, SW4 KEYSW, SW40 KEYSW, SW41 KEYSW, SW42 KEYSW, SW43 KEYSW, SW44 KEYSW, SW45 KEYSW, SW46 KEYSW, SW47 KEYSW, SW48 KEYSW, SW49 KEYSW, SW5 KEYSW, SW50 KEYSW, SW51 KEYSW, SW52 KEYSW, SW53 KEYSW, SW54 KEYSW, SW55 KEYSW, SW56 KEYSW, SW57 KEYSW, SW58 KEYSW, SW59 KEYSW, SW6 KEYSW, SW60 KEYSW, SW61 KEYSW, SW62 KEYSW, SW63 KEYSW, SW64 KEYSW, SW65 KEYSW, SW66 KEYSW, SW67 KEYSW, SW68 KEYSW, SW69 KEYSW, SW7 KEYSW, SW70 KEYSW, SW71 KEYSW, SW72 KEYSW, SW73 KEYSW, SW74 KEYSW, SW75 KEYSW, SW8 KEYSW, SW9 KEYSW, U1 ATmega32A-PU, Y1 Crystal

Commit message: fixed some footprints and removed switch options
Parts:
- removed ST72: 7U, cftkb:MX-7U-Stabilizer
- removed SW31: KEYSW, cftkb:SW_Cherry_MX1A_1.75u_PCBNOSCREEN
- removed SW43, SW45: KEYSW, cftkb:SW_Cherry_MX1A_2.25u_PCBNOSCREEN
- removed SW70, SW71, SW73, SW74: KEYSW, cftkb:SW_Cherry_MX1A_1.50u_PCBNOSCREEN
- removed SW72: KEYSW, cftkb:SW_Cherry_MX1A_1.00u_PCB-NOSCREEN
- removed SWb29: KEYSW, MX_Only:MXOnly-ISO-ROTATED-ReversedStabilizers-NoLED
- C1, C2: footprint cftkb:D_DO-35_SOD27_P5.08mm_Horizontal -> Capacitor_THT:C_Disc_D3.4mm_W2.1mm_P2.50mm
- C3: footprint cftkb:D_DO-35_SOD27_P5.08mm_Horizontal -> Capacitor_THT:CP_Radial_D4.0mm_P1.50mm
- C4, C5: footprint cftkb:D_DO-35_SOD27_P5.08mm_Horizontal -> Capacitor_THT:C_Disc_D5.0mm_W2.5mm_P5.00mm
- SW29: footprint cftkb:SW_Cherry_MX1A_1.50u_PCBNOSCREEN -> cftkb:SW_Cherry_MX1A_2.00u_PCBNOSCREEN
- moved SW29 17.9 mm to (339.5, 121.2), turned to 270 degrees
- moved C2 0.06 mm to (334.5, 77.3)
Routing:
- net Net-(D62-Pad2): track 355.8 -> 337.9 mm
- net Net-(D61-Pad2): track 425.1 -> 408.5 mm
- net col10: track 251.0 -> 236.7 mm
- net col2: track 329.2 -> 316.6 mm
- net Net-(D29-Pad2): track 139.3 -> 128.9 mm
- net Net-(D59-Pad2): track 462.2 -> 453.3 mm
- net col6: track 279.4 -> 273.7 mm
- net col0: track 364.5 -> 359.2 mm
- net Net-(D63-Pad2): track 279.4 -> 274.6 mm
- net col13: track 162.0 -> 165.6 mm
- net GND: track 241.1 -> 238.9 mm
- net Net-(D43-Pad2): track 152.5 -> 150.5 mm, vias 0 -> 1
- net Net-(D56-Pad2): track 147.3 -> 145.7 mm
Other:
- board text removed: "1.25U"
- board text removed: "1.5U"
- board text removed: "1U"
- board text removed: "STANDARD"
- board text removed: "STEPPED"

Commit message: ignore file updated
Routing:
- net col0: track 359.2 -> 341.8 mm
- net GND: vias 36 -> 35
Changed lines of the file:
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@@
     (thickness 1.6)
     (drawings 28)
-    (tracks 2207)
+    (tracks 2200)
     (zones 0)
     (modules 175)
@@
   (via (at 311.633443 61.364317) (size 0.8) (drill 0.4) (layers F.Cu B.Cu) (net 1))
   (via (at 309.078784 61.364317) (size 0.8) (drill 0.4) (layers F.Cu B.Cu) (net 1))
-  (via (at 295.115646 55.747566) (size 0.8) (drill 0.4) (layers F.Cu B.Cu) (net 1))
   (via (at 331.04 87.5) (size 0.8) (drill 0.4) (layers F.Cu B.Cu) (net 1))
   (segment (start 282.195002 61.633652) (end 282.200002 61.638652) (width 0.4) (layer F.Cu) (net 2))
@@
   (segment (start 77.420284 103.99138) (end 77.420284 120.66008) (width 0.25) (layer B.Cu) (net 75))
   (segment (start 75.042915 161.137449) (end 75.038984 161.14138) (width 0.25) (layer B.Cu) (net 75))
-  (segment (start 77.420234 161.137449) (end 75.042915 161.137449) (width 0.25) (layer B.Cu) (net 75))
-  (segment (start 84.563984 151.426244) (end 84.563984 158.026306) (width 0.25) (layer B.Cu) (net 75))
-  (segment (start 84.563984 142.09138) (end 84.563984 151.426244) (width 0.25) (layer B.Cu) (net 75))
-  (segment (start 84.563984 151.426244) (end 84.563984 151.61638) (width 0.25) (layer B.Cu) (net 75))
-  (segment (start 81.452841 161.137449) (end 77.420234 161.137449) (width 0.25) (layer B.Cu) (net 75))
-  (segment (start 84.563984 158.026306) (end 81.452841 161.137449) (width 0.25) (layer B.Cu) (net 75))
   (segment (start 312.881738 57.668586) (end 311.609964 56.396812) (width 0.25) (layer B.Cu) (net 75))
   (segment (start 72.657784 84.94138) (end 72.657784 83.385746) (width 0.25) (layer B.Cu) (net 75))
@@
   (segment (start 312.881738 71.969274) (end 312.881738 57.668586) (width 0.25) (layer B.Cu) (net 75))
   (segment (start 312.089199 72.761813) (end 312.881738 71.969274) (width 0.25) (layer B.Cu) (net 75))
-  (segment (start 84.560204 142.0876) (end 84.563984 142.09138) (width 0.25) (layer B.Cu) (net 75))
-  (segment (start 75.0316 142.0876) (end 84.560204 142.0876) (width 0.25) (layer B.Cu) (net 75))
   (segment (start 75.039034 142.080166) (end 75.0316 142.0876) (width 0.25) (layer B.Cu) (net 75))
   (segment (start 75.039034 123.03125) (end 75.039034 142.080166) (width 0.25) (layer B.Cu) (net 75))
   (segment (start 77.410204 120.66008) (end 77.420284 120.66008) (width 0.25) (layer B.Cu) (net 75))
   (segment (start 75.039034 123.03125) (end 77.410204 120.66008) (width 0.25) (layer B.Cu) (net 75))
+  (segment (start 75.0316 161.123866) (end 75.038984 161.13125) (width 0.25) (layer B.Cu) (net 75))
+  (segment (start 75.0316 142.0876) (end 75.0316 161.123866) (width 0.25) (layer B.Cu) (net 75))
   (segment (start 91.707784 94.46638) (end 101.232784 103.99138) (width 0.25) (layer B.Cu) (net 76))
   (segment (start 91.707784 84.94138) (end 91.707784 94.46638) (width 0.25) (layer B.Cu) (net 76))
